File: rs485.kicad_sch (KiCad schematic)
At the start: 3 parts, among them J17 TermBlock-3P-381, U8 ADM3485E

Commit message: Populate module/purpose fields for BOM, generate iBOM
Parts:
- C?, J17, U8: SternDMX yes -> (none)
Changed lines of the file:
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@@
-      (effects (font (size 1.27 1.27)) hide)
-    )
-    (property "HAVAS" "" (at 176.53 100.33 0)
       (effects (font (size 1.27 1.27)) hide)
     )
@@
     )
     (property "Purpose" "Line Driver" (at 176.53 100.33 0)
-      (effects (font (size 1.27 1.27)) hide)
-    )
-    (property "SternDMX" "yes" (at 176.53 100.33 0)
-      (effects (font (size 1.27 1.27)) hide)
-    )
-    (property "SternPult" "" (at 176.53 100.33 0)
       (effects (font (size 1.27 1.27)) hide)
     )
@@
       (effects (font (size 1.27 1.27)) hide)
     )
-    (property "HAVAS" "" (at 153.67 91.44 0)
-      (effects (font (size 1.27 1.27)) hide)
-    )
     (property "Module" "RS485" (at 153.67 91.44 0)
       (effects (font (size 1.27 1.27)) hide)
     )
     (property "Purpose" "ADM3485E bulk cap" (at 153.67 91.44 0)
-      (effects (font (size 1.27 1.27)) hide)
-    )
-    (property "SternDMX" "yes" (at 153.67 91.44 0)
-      (effects (font (size 1.27 1.27)) hide)
-    )
-    (property "SternPult" "" (at 153.67 91.44 0)
       (effects (font (size 1.27 1.27)) hide)
     )
@@
       (effects (font (size 1.27 1.27)) hide)
     )
-    (property "HAVAS" "" (at 106.68 104.14 0)
-      (effects (font (size 1.27 1.27)) hide)
-    )
     (property "Module" "RS485" (at 106.68 104.14 0)
       (effects (font (size 1.27 1.27)) hide)
     )
-    (property "SternDMX" "yes" (at 106.68 104.14 0)
-      (effects (font (size 1.27 1.27)) hide)
-    )
-    (property "SternPult" "" (at 106.68 104.14 0)
-      (effects (font (size 1.27 1.27)) hide)
-    )
