File: omega2ethernet.kicad_sch (KiCad schematic)
At the start: 11 parts, among them J11 Pulse-J0026D21B

Commit message: schematic DRC now ok
Connections:
- net +3V3 renamed +3.3V

Commit message: Populate module/purpose fields for BOM, generate iBOM
Parts:
- C13, C14, C15: Module (none) -> Ethernet; Purpose (none) -> Termination
- C16: Module (none) -> Ethernet; Purpose (none) -> RJ45 Shield HF Conn
- J11, R10, R11, R12, R9: Module (none) -> Ethernet
- R7, R8: Module (none) -> Ethernet LED
Changed lines of the file:
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@@
+      (effects (font (size 1.27 1.27)) hide)
+    )
+    (property "Module" "Ethernet" (at 120.65 125.73 0)
+      (effects (font (size 1.27 1.27)) hide)
+    )
+    (property "Purpose" "Termination" (at 120.65 125.73 0)
       (effects (font (size 1.27 1.27)) hide)
     )
@@
       (effects (font (size 1.27 1.27)) hide)
     )
+    (property "Module" "Ethernet" (at 105.41 67.31 0)
+      (effects (font (size 1.27 1.27)) hide)
+    )
     (pin "1")
     (pin "2")
@@
       (effects (font (size 1.27 1.27)) hide)
     )
+    (property "Module" "Ethernet" (at 109.22 67.31 0)
+      (effects (font (size 1.27 1.27)) hide)
+    )
     (pin "1")
     (pin "2")
@@
       (effects (font (size 1.27 1.27)) hide)
     )
+    (property "Module" "Ethernet" (at 113.03 67.31 0)
+      (effects (font (size 1.27 1.27)) hide)
+    )
     (pin "1")
     (pin "2")
@@
     )
     (property "Manufacturer" "RND" (at 116.84 67.31 0)
+      (effects (font (size 1.27 1.27)) hide)
+    )
+    (property "Module" "Ethernet" (at 116.84 67.31 0)
       (effects (font (size 1.27 1.27)) hide)
     )
@@
       (effects (font (size 1.27 1.27)) hide)
     )
+    (property "Module" "Ethernet" (at 95.25 67.31 0)
+      (effects (font (size 1.27 1.27)) hide)
+    )
+    (property "Purpose" "Termination" (at 95.25 67.31 0)
+      (effects (font (size 1.27 1.27)) hide)
+    )
     (pin "1")
     (pin "2")
@@
       (effects (font (size 1.27 1.27)) hide)
     )
+    (property "Module" "Ethernet" (at 127 67.31 0)
+      (effects (font (size 1.27 1.27)) hide)
+    )
+    (property "Purpose" "Termination" (at 127 67.31 0)
+      (effects (font (size 1.27 1.27)) hide)
+    )
     (pin "1")
     (pin "2")
@@
       (effects (font (size 1.27 1.27)))
     )
-    (property "Field4" "" (at 101.6 115.57 90)
-      (effects (font (size 1.524 1.524)) hide)
-    )
-    (property "Field5" "" (at 101.6 115.57 90)
-      (effects (font (size 1.524 1.524)) hide)
-    )
     (property "Vendor" "distrelec.ch" (at 101.6 115.57 0)
       (effects (font (size 1.27 1.27)) hide)
@@
       (effects (font (size 1.27 1.27)) hide)
     )
+    (property "Module" "Ethernet LED" (at 101.6 115.57 0)
+      (effects (font (size 1.27 1.27)) hide)
+    )
     (pin "1")
     (pin "2")
@@
     )
     (property "Vendor" "distrelec.ch" (at 101.6 120.65 0)
+      (effects (font (size 1.27 1.27)) hide)
+    )
+    (property "Module" "Ethernet LED" (at 101.6 120.65 0)
       (effects (font (size 1.27 1.27)) hide)
     )
@@
       (effects (font (size 1.524 1.524)) hide)
     )
-    (property "Field4" "" (at 154.94 101.6 0)
-      (effects (font (size 1.524 1.524)) hide)
-    )
-    (property "Field5" "" (at 154.94 101.6 0)
-      (effects (font (size 1.524 1.524)) hide)
-    )
     (property "MPN" "J0026D21B" (at 154.94 101.6 0)
       (effects (font (size 1.27 1.27)) hide)
     )
     (property "Vendor" "Fundus S.Flüeler" (at 154.94 101.6 0)
+      (effects (font (size 1.27 1.27)) hide)
+    )
+    (property "Module" "Ethernet" (at 154.94 101.6 0)
       (effects (font (size 1.27 1.27)) hide)
     )
@@
       (effects (font (size 1.27 1.27)))
     )
-    (property "Field4" "" (at 160.02 125.73 0)
-      (effects (font (size 1.524 1.524)) hide)
-    )
-    (property "Field5" "" (at 160.02 125.73 0)
-      (effects (font (size 1.524 1.524)) hide)
-    )
     (property "SKU" "301-11-186" (at 160.02 125.73 0)
       (effects (font (size 1.27 1.27)) hide)
@@
       (effects (font (size 1.27 1.27)) hide)
     )
+    (property "Module" "Ethernet" (at 160.02 125.73 0)
+      (effects (font (size 1.27 1.27)) hide)
+    )
+    (property "Purpose" "RJ45 Shield HF Conn" (at 160.02 125.73 0)
+      (effects (font (size 1.27 1.27)) hide)
+    )

Commit message: Adjustments for BOM
Parts:
- J11: Purpose (none) -> RJ45 Jack
Changed lines of the file:
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@@
+      (effects (font (size 1.27 1.27)) hide)
+    )
+    (property "Purpose" "RJ45 Jack" (at 154.94 101.6 0)
       (effects (font (size 1.27 1.27)) hide)
     )
